Commit message: Imported upstream version '3.0.0' of 'upstream'

File: gazebo/gazebo.urdf.xacro (robot description, xacro)
@@ -1,11 +1,20 @@
 <?xml version="1.0"?>
 <!--
-  Copyright (c) 2011, PAL Robotics, S.L.
-  All rights reserved.
-  This work is licensed under the Creative Commons Attribution-NonCommercial-NoDerivs 3.0 Unported License.
-  To view a copy of this license, visit http://creativecommons.org/licenses/by-nc-nd/3.0/ or send a letter to
-  Creative Commons, 444 Castro Street, Suite 900, Mountain View, California, 94041, USA.
--->
+Copyright (c) 2022 PAL Robotics S.L. All rights reserved.
+Licensed under the Apache License, Version 2.0 (the "License");
+you may not use this file except in compliance with the License.
+You may obtain a copy of the License at
+    http://www.apache.org/licenses/LICENSE-2.0
+Unless required by applicable law or agreed to in writing, software
+distributed under the License is distributed on an "AS IS" BASIS,
+WITHOUT WARRANTIES OR CONDITIONS OF ANY KIND, either express or implied.
+See the License for the specific language governing permissions and
+limitations under the License.
+ -->
 <robot xmlns:xacro="http://ros.org/wiki/xacro">
+   <xacro:arg name="multiple" default="false"/>
+   <xacro:arg name="namespace" default=""/>
+   <xacro:property name="is_multiple" value="$(arg multiple)" />
+   <xacro:property name="nsp" value="$(arg namespace)" />
    <xacro:macro name="hey5_gazebo_simulation" params="side">
    <gazebo>
@@ -15,21 +24,59 @@
         <name>${side}_thumb_abd_joint</name>
         <scale_factor>2.0</scale_factor>
+	<pid_gains>
+	  <p>50</p>
+	  <i>0.1</i>
+	  <d>0.1</d>
+	  <i_max>1</i_max>
+	  <i_min>-1</i_min>
+	</pid_gains>
       </virtualJoint>
       <virtualJoint>
         <name>${side}_thumb_flex_1_joint</name>
         <scale_factor>2.5</scale_factor>
+	<pid_gains>
+	  <p>50</p>
+	  <i>0.1</i>
+	  <d>0.1</d>
+	  <i_max>1</i_max>
+	  <i_min>-1</i_min>
+	</pid_gains>
       </virtualJoint>
       <virtualJoint>
         <name>${side}_thumb_virtual_1_joint</name>
         <scale_factor>3.0</scale_factor>
+	<pid_gains>
+	  <p>50</p>
+	  <i>0.1</i>
+	  <d>0.1</d>
+	  <i_max>1</i_max>
+	  <i_min>-1</i_min>
+	</pid_gains>
       </virtualJoint>
       <virtualJoint>
         <name>${side}_thumb_flex_2_joint</name>
         <scale_factor>3.5</scale_factor>
+	<pid_gains>
+	  <p>50</p>
+	  <i>0.1</i>
+	  <d>0.1</d>
+	  <i_max>1</i_max>
+	  <i_min>-1</i_min>
+	</pid_gains>
       </virtualJoint>
       <virtualJoint>
         <name>${side}_thumb_virtual_2_joint</name>
         <scale_factor>3.0</scale_factor>
-      </virtualJoint>
+	<pid_gains>
+	  <p>50</p>
+	  <i>0.1</i>
+	  <d>0.1</d>
+	  <i_max>1</i_max>
+	  <i_min>-1</i_min>
+	</pid_gains>
+      </virtualJoint>
+      <xacro:if value="${is_multiple}">
+          <robotNamespace>/${nsp}</robotNamespace>
+      </xacro:if>
     </plugin>
     <plugin filename="libgazebo_underactuated_finger.so" name="gazebo_${side}_index">
@@ -38,25 +85,70 @@
         <name>${side}_index_abd_joint</name>
         <scale_factor>5.0</scale_factor>
+	<pid_gains>
+	  <p>50</p>
+	  <i>0.1</i>
+	  <d>0.1</d>
+	  <i_max>1</i_max>
+	  <i_min>-1</i_min>
+	</pid_gains>
       </virtualJoint>
       <virtualJoint>
         <name>${side}_index_flex_1_joint</name>
         <scale_factor>2.5</scale_factor>
+	<pid_gains>
+	  <p>50</p>
+	  <i>0.1</i>
+	  <d>0.1</d>
+	  <i_max>1</i_max>
+	  <i_min>-1</i_min>
+	</pid_gains>
       </virtualJoint>
       <virtualJoint>
         <name>${side}_index_virtual_1_joint</name>
         <scale_factor>3.0</scale_factor>
+	<pid_gains>
+	  <p>50</p>
+	  <i>0.1</i>
+	  <d>0.1</d>
+	  <i_max>1</i_max>
+	  <i_min>-1</i_min>
+	</pid_gains>
       </virtualJoint>
       <virtualJoint>
         <name>${side}_index_flex_2_joint</name>
         <scale_factor>3.5</scale_factor>
+	<pid_gains>
+	  <p>50</p>
+	  <i>0.1</i>
+	  <d>0.1</d>
+	  <i_max>1</i_max>
+	  <i_min>-1</i_min>
+	</pid_gains>
       </virtualJoint>
       <virtualJoint>
         <name>${side}_index_virtual_2_joint</name>
         <scale_factor>3.5</scale_factor>
+	<pid_gains>
+	  <p>50</p>
+	  <i>0.1</i>
+	  <d>0.1</d>
+	  <i_max>1</i_max>
+	  <i_min>-1</i_min>
+	</pid_gains>
       </virtualJoint>
       <virtualJoint>
         <name>${side}_index_flex_3_joint</name>
         <scale_factor>4.0</scale_factor>
-      </virtualJoint>
+	<pid_gains>
+	  <p>50</p>
+	  <i>0.1</i>
+	  <d>0.1</d>
+	  <i_max>1</i_max>
+	  <i_min>-1</i_min>
+	</pid_gains>
+      </virtualJoint>
+      <xacro:if value="${is_multiple}">
+          <robotNamespace>/${nsp}</robotNamespace>
+      </xacro:if>
     </plugin>
     <plugin filename="libgazebo_underactuated_finger.so" name="gazebo_${side}_middle">
@@ -65,21 +157,59 @@
         <name>${side}_middle_flex_1_joint</name>
         <scale_factor>2.5</scale_factor>
+	<pid_gains>
+	  <p>50</p>
+	  <i>0.1</i>
+	  <d>0.1</d>
+	  <i_max>1</i_max>
+	  <i_min>-1</i_min>
+	</pid_gains>
       </virtualJoint>
       <virtualJoint>
         <name>${side}_middle_virtual_1_joint</name>
         <scale_factor>3.0</scale_factor>
+	<pid_gains>
+	  <p>50</p>
+	  <i>0.1</i>
+	  <d>0.1</d>
+	  <i_max>1</i_max>
+	  <i_min>-1</i_min>
+	</pid_gains>
       </virtualJoint>
       <virtualJoint>
         <name>${side}_middle_flex_2_joint</name>
         <scale_factor>3.5</scale_factor>
+	<pid_gains>
+	  <p>50</p>
+	  <i>0.1</i>
+	  <d>0.1</d>
+	  <i_max>1</i_max>
+	  <i_min>-1</i_min>
+	</pid_gains>
       </virtualJoint>
       <virtualJoint>
         <name>${side}_middle_virtual_2_joint</name>
         <scale_factor>3.5</scale_factor>
+	<pid_gains>
+	  <p>50</p>
+	  <i>0.1</i>
+	  <d>0.1</d>
+	  <i_max>1</i_max>
+	  <i_min>-1</i_min>
+	</pid_gains>
       </virtualJoint>
       <virtualJoint>
         <name>${side}_middle_flex_3_joint</name>
         <scale_factor>4.0</scale_factor>
-      </virtualJoint>
+	<pid_gains>
+	  <p>50</p>
+	  <i>0.1</i>
+	  <d>0.1</d>
+	  <i_max>1</i_max>
+	  <i_min>-1</i_min>
+	</pid_gains>
+      </virtualJoint>
+      <xacro:if value="${is_multiple}">
+          <robotNamespace>/${nsp}</robotNamespace>
+      </xacro:if>
     </plugin>
     <plugin filename="libgazebo_underactuated_finger.so" name="gazebo_${side}_ring">
@@ -88,21 +218,59 @@
         <name>${side}_ring_flex_1_joint</name>
         <scale_factor>2.5</scale_factor>
+	<pid_gains>
+	  <p>50</p>
+	  <i>0.1</i>
+	  <d>0.1</d>
+	  <i_max>1</i_max>
+	  <i_min>-1</i_min>
+	</pid_gains>
       </virtualJoint>
       <virtualJoint>
         <name>${side}_ring_virtual_1_joint</name>
         <scale_factor>3.0</scale_factor>
+	<pid_gains>
+	  <p>50</p>
+	  <i>0.1</i>
+	  <d>0.1</d>
+	  <i_max>1</i_max>
+	  <i_min>-1</i_min>
+	</pid_gains>
       </virtualJoint>
       <virtualJoint>
         <name>${side}_ring_flex_2_joint</name>
         <scale_factor>3.5</scale_factor>
+	<pid_gains>
+	  <p>50</p>
+	  <i>0.1</i>
+	  <d>0.1</d>
+	  <i_max>1</i_max>
+	  <i_min>-1</i_min>
+	</pid_gains>
       </virtualJoint>
       <virtualJoint>
         <name>${side}_ring_virtual_2_joint</name>
         <scale_factor>3.5</scale_factor>
+	<pid_gains>
+	  <p>50</p>
+	  <i>0.1</i>
+	  <d>0.1</d>
+	  <i_max>1</i_max>
+	  <i_min>-1</i_min>
+	</pid_gains>
       </virtualJoint>
       <virtualJoint>
         <name>${side}_ring_flex_3_joint</name>
         <scale_factor>4.0</scale_factor>
-      </virtualJoint>
+	<pid_gains>
+	  <p>50</p>
+	  <i>0.1</i>
+	  <d>0.1</d>
+	  <i_max>1</i_max>
+	  <i_min>-1</i_min>
+	</pid_gains>
+      </virtualJoint>
+      <xacro:if value="${is_multiple}">
+          <robotNamespace>/${nsp}</robotNamespace>
+      </xacro:if>
     </plugin>
     <plugin filename="libgazebo_underactuated_finger.so" name="gazebo_${side}_little">
@@ -111,21 +279,59 @@
         <name>${side}_little_flex_1_joint</name>
         <scale_factor>2.5</scale_factor>
+	<pid_gains>
+	  <p>50</p>
+	  <i>0.1</i>
+	  <d>0.1</d>
+	  <i_max>1</i_max>
+	  <i_min>-1</i_min>
+	</pid_gains>
       </virtualJoint>
       <virtualJoint>
         <name>${side}_little_virtual_1_joint</name>
         <scale_factor>3.0</scale_factor>
+	<pid_gains>
+	  <p>50</p>
+	  <i>0.1</i>
+	  <d>0.1</d>
+	  <i_max>1</i_max>
+	  <i_min>-1</i_min>
+	</pid_gains>
       </virtualJoint>
       <virtualJoint>
         <name>${side}_little_flex_2_joint</name>
         <scale_factor>3.5</scale_factor>
+	<pid_gains>
+	  <p>50</p>
+	  <i>0.1</i>
+	  <d>0.1</d>
+	  <i_max>1</i_max>
+	  <i_min>-1</i_min>
+	</pid_gains>
       </virtualJoint>
       <virtualJoint>
         <name>${side}_little_virtual_2_joint</name>
         <scale_factor>3.5</scale_factor>
+	<pid_gains>
+	  <p>50</p>
+	  <i>0.1</i>
+	  <d>0.1</d>
+	  <i_max>1</i_max>
+	  <i_min>-1</i_min>
+	</pid_gains>
       </virtualJoint>
       <virtualJoint>
         <name>${side}_little_flex_3_joint</name>
         <scale_factor>4.0</scale_factor>
-      </virtualJoint>
+	<pid_gains>
+	  <p>50</p>
+	  <i>0.1</i>
+	  <d>0.1</d>
+	  <i_max>1</i_max>
+	  <i_min>-1</i_min>
+	</pid_gains>
+      </virtualJoint>
+      <xacro:if value="${is_multiple}">
+          <robotNamespace>/${nsp}</robotNamespace>
+      </xacro:if>
     </plugin>
   </gazebo>

File: robots/hey5_test.urdf.xacro (robot description, xacro)
@@ -1,10 +1,15 @@
 <?xml version="1.0"?>
 <!--
-  Copyright (c) 2014, PAL Robotics, S.L.
-  All rights reserved.
-  This work is licensed under the Creative Commons Attribution-NonCommercial-NoDerivs 3.0 Unported License.
-  To view a copy of this license, visit http://creativecommons.org/licenses/by-nc-nd/3.0/ or send a letter to
-  Creative Commons, 444 Castro Street, Suite 900, Mountain View, California, 94041, USA.
--->
+Copyright (c) 2022 PAL Robotics S.L. All rights reserved.
+Licensed under the Apache License, Version 2.0 (the "License");
+you may not use this file except in compliance with the License.
+You may obtain a copy of the License at
+    http://www.apache.org/licenses/LICENSE-2.0
+Unless required by applicable law or agreed to in writing, software
+distributed under the License is distributed on an "AS IS" BASIS,
+WITHOUT WARRANTIES OR CONDITIONS OF ANY KIND, either express or implied.
+See the License for the specific language governing permissions and
+limitations under the License.
+ -->
 <robot xmlns:xacro="http://ros.org/wiki/xacro"
        name="hey5">

File: urdf/actuators.urdf.xacro (robot description, xacro)
@@ -1,16 +1,21 @@
 <?xml version="1.0"?>
 <!--
-  Copyright (c) 2014, PAL Robotics, S.L.
-  All rights reserved.
-  This work is licensed under the Creative Commons Attribution 4.0 International License.
-  To view a copy of this license, visit http://creativecommons.org/licenses/by/4.0 or send a letter to
-  Creative Commons, 444 Castro Street, Suite 900, Mountain View, California, 94041, USA.
--->
+Copyright (c) 2022 PAL Robotics S.L. All rights reserved.
+Licensed under the Apache License, Version 2.0 (the "License");
+you may not use this file except in compliance with the License.
+You may obtain a copy of the License at
+    http://www.apache.org/licenses/LICENSE-2.0
+Unless required by applicable law or agreed to in writing, software
+distributed under the License is distributed on an "AS IS" BASIS,
+WITHOUT WARRANTIES OR CONDITIONS OF ANY KIND, either express or implied.
+See the License for the specific language governing permissions and
+limitations under the License.
+ -->
 <robot xmlns:xacro="http://ros.org/wiki/xacro">
   <!-- Thumb actuator -->
   <xacro:macro name="thumb_actuator" params="name parent *origin">
     <xacro:actuator_impl parent="${parent}" name="${name}">
-      <insert_block name="origin" />
-      <limit lower="${-150 * deg_to_rad}" upper="${360 * deg_to_rad}" effort="2.0" velocity="3.35" /> <!-- TODO: Tune effort -->
+      <xacro:insert_block name="origin" />
+      <limit lower="${-150 * deg_to_rad}" upper="${360 * deg_to_rad}" effort="2.0" velocity="3.35" />
       <safety_controller k_position="20"
                          k_velocity="20"
@@ -22,6 +27,6 @@
   <xacro:macro name="index_actuator" params="name parent *origin">
     <xacro:actuator_impl parent="${parent}" name="${name}">
-      <insert_block name="origin" />
-      <limit lower="${-175 * deg_to_rad}" upper="${390 * deg_to_rad}" effort="2.0" velocity="3.35" /> <!-- TODO: Tune effort -->
+      <xacro:insert_block name="origin" />
+      <limit lower="${-175 * deg_to_rad}" upper="${390 * deg_to_rad}" effort="2.0" velocity="3.35" />
       <safety_controller k_position="20"
                          k_velocity="20"
@@ -33,6 +38,6 @@
   <xacro:macro name="mrl_actuator" params="name parent *origin">
     <xacro:actuator_impl parent="${parent}" name="${name}">
-      <insert_block name="origin" />
-      <limit lower="${-145 * deg_to_rad}" upper="${530 * deg_to_rad}" effort="2.0" velocity="3.56" /> <!-- TODO: Tune effort -->
+      <xacro:insert_block name="origin" />
+      <limit lower="${-145 * deg_to_rad}" upper="${530 * deg_to_rad}" effort="2.0" velocity="3.56" />
       <safety_controller k_position="20"
                          k_velocity="20"
@@ -54,9 +59,9 @@
       <parent link="${parent}" />
       <child link="${name}_link" />
-      <insert_block name="origin" />
+      <xacro:insert_block name="origin" />
       <axis xyz="0 0 1" />
-      <insert_block name="limit" />
-      <dynamics friction="0.0" damping="0.5"/> <!-- TODO: Tune -->
-      <insert_block name="safety_controller" />
+      <xacro:insert_block name="limit" />
+      <dynamics friction="0.0" damping="0.5"/>
+      <xacro:insert_block name="safety_controller" />
     </joint>
     <link name="${name}_link">

File: urdf/deg_to_rad.urdf.xacro (robot description, xacro)
@@ -1,11 +1,16 @@
 <?xml version="1.0"?>
 <!--
-  Copyright (c) 2011, PAL Robotics, S.L.
-  All rights reserved.
-  This work is licensed under the Creative Commons Attribution 4.0 International License.
-  To view a copy of this license, visit http://creativecommons.org/licenses/by/4.0 or send a letter to
-  Creative Commons, 444 Castro Street, Suite 900, Mountain View, California, 94041, USA.
--->
+Copyright (c) 2022 PAL Robotics S.L. All rights reserved.
+Licensed under the Apache License, Version 2.0 (the "License");
+you may not use this file except in compliance with the License.
+You may obtain a copy of the License at
+    http://www.apache.org/licenses/LICENSE-2.0
+Unless required by applicable law or agreed to in writing, software
+distributed under the License is distributed on an "AS IS" BASIS,
+WITHOUT WARRANTIES OR CONDITIONS OF ANY KIND, either express or implied.
+See the License for the specific language governing permissions and
+limitations under the License.
+ -->
 <robot xmlns:xacro="http://ros.org/wiki/xacro">
-  <property name="deg_to_rad" value="0.01745329251994329577" />
+  <xacro:property name="deg_to_rad" value="0.01745329251994329577" />
 </robot>

File: urdf/fingers.urdf.xacro (robot description, xacro)
@@ -1,10 +1,15 @@
 <?xml version="1.0"?>
 <!--
-  Copyright (c) 2014, PAL Robotics, S.L.
-  All rights reserved.
-  This work is licensed under the Creative Commons Attribution 4.0 International License.
-  To view a copy of this license, visit http://creativecommons.org/licenses/by/4.0 or send a letter to
-  Creative Commons, 444 Castro Street, Suite 900, Mountain View, California, 94041, USA.
--->
+Copyright (c) 2022 PAL Robotics S.L. All rights reserved.
+Licensed under the Apache License, Version 2.0 (the "License");
+you may not use this file except in compliance with the License.
+You may obtain a copy of the License at
+    http://www.apache.org/licenses/LICENSE-2.0
+Unless required by applicable law or agreed to in writing, software
+distributed under the License is distributed on an "AS IS" BASIS,
+WITHOUT WARRANTIES OR CONDITIONS OF ANY KIND, either express or implied.
+See the License for the specific language governing permissions and
+limitations under the License.
+ -->
 <robot xmlns:xacro="http://ros.org/wiki/xacro">
   <!--External resources-->
@@ -14,12 +19,12 @@
   <xacro:property name="thumb_abd_min"   value="${  0 * deg_to_rad}" />
   <xacro:property name="thumb_abd_max"   value="${ 90 * deg_to_rad}" />
-  <xacro:property name="finger_abd_min"  value="${-30 * deg_to_rad}" /> <!--TODO: Check-->
-  <xacro:property name="finger_abd_max"  value="${ 30 * deg_to_rad}" /> <!--TODO: Check-->
+  <xacro:property name="finger_abd_min"  value="${-30 * deg_to_rad}" />
+  <xacro:property name="finger_abd_max"  value="${ 30 * deg_to_rad}" />
   <xacro:property name="finger_flex_min" value="${  0 * deg_to_rad}" />
   <xacro:property name="finger_flex_max" value="${ 45 * deg_to_rad}" />
-  <xacro:property name="finger_max_vel"  value="2.0" />                 <!--TODO: Check-->
-  <xacro:property name="finger_max_eff"  value="2.0" />                 <!--TODO: Check-->
-  <xacro:property name="finger_friction" value="0.0" />                 <!--TODO: Check-->
-  <xacro:property name="finger_damping"  value="0.5" />                 <!--TODO: Check-->
+  <xacro:property name="finger_max_vel"  value="2.0" />
+  <xacro:property name="finger_max_eff"  value="2.0" />
+  <xacro:property name="finger_friction" value="0.0" />
+  <xacro:property name="finger_damping"  value="0.5" />
   <xacro:property name="finger_d1"  value="0.009" />
   <xacro:property name="finger_d2"  value="0.013" />
@@ -41,5 +46,5 @@
     <!--Abductor-->
     <xacro:finger_abd parent="${parent}" name="${name}_abd" reflect="${reflect}">
-      <insert_block name="origin" />
+      <xacro:insert_block name="origin" />
     </xacro:finger_abd>
     <!--First flexor-->
@@ -77,5 +82,5 @@
     <!--Abductor-->
     <xacro:thumb_abd parent="${parent}" name="${name}_abd" reflect="${reflect}">
-      <insert_block name="origin" />
+      <xacro:insert_block name="origin" />
     </xacro:thumb_abd>
     <!--First flexor-->
@@ -106,5 +111,5 @@
       <parent link="${parent}" />
       <child link="${name}_link" />
-      <insert_block name="origin" />
+      <xacro:insert_block name="origin" />
       <axis xyz="0 0 1" />
       <limit lower="${finger_abd_min}" upper="${finger_abd_max}" effort="${finger_max_eff}" velocity="${finger_max_vel}" />
@@ -147,5 +152,5 @@
       <parent link="${parent}" />
       <child link="${name}_link" />
-      <insert_block name="origin" />
+      <xacro:insert_block name="origin" />
       <axis xyz="0 0 1" />
       <limit lower="${thumb_abd_min}" upper="${thumb_abd_max}" effort="${finger_max_eff}" velocity="${finger_max_vel}" />
@@ -189,5 +194,5 @@
       <parent link="${parent}" />
       <child link="${name}_link" />
-      <insert_block name="origin" />
+      <xacro:insert_block name="origin" />
       <axis xyz="0 0 1" />
       <limit lower="${finger_flex_min}" upper="${finger_flex_max}" effort="${finger_max_eff}" velocity="${finger_max_vel}" />
@@ -197,5 +202,5 @@
       <inertial>
         <origin xyz="${finger_d2 / 2.0} 0 0" rpy="0 0 0" />
-        <mass value="0.01" /> <!--TODO: can we make it zero and still have a stable dynamic simulation?-->
+        <mass value="0.01" />
         <inertia ixx="0.001" ixy="0" ixz="0" iyy="0.001" iyz="0" izz="0.001" /> <!-- To stabilize simulation -->
       </inertial>
@@ -232,5 +237,5 @@
       <parent link="${parent}" />
       <child link="${name}_link" />
-      <insert_block name="origin" />
+      <xacro:insert_block name="origin" />
       <axis xyz="0 0 1" />
       <limit lower="${finger_flex_min}" upper="${finger_flex_max}" effort="${finger_max_eff}" velocity="${finger_max_vel}" />
@@ -275,5 +280,5 @@
       <parent link="${parent}" />
       <child link="${name}_link" />
-      <insert_block name="origin" />
+      <xacro:insert_block name="origin" />
       <axis xyz="0 0 1" />
       <limit lower="${finger_flex_min}" upper="${finger_flex_max}" effort="${finger_max_eff}" velocity="${finger_max_vel}" />

File: urdf/hey5_hand.urdf.xacro (robot description, xacro)
@@ -1,10 +1,15 @@
 <?xml version="1.0"?>
 <!--
-  Copyright (c) 2014, PAL Robotics, S.L.
-  All rights reserved.
-  This work is licensed under the Creative Commons Attribution 4.0 International License.
-  To view a copy of this license, visit http://creativecommons.org/licenses/by/4.0 or send a letter to
-  Creative Commons, 444 Castro Street, Suite 900, Mountain View, California, 94041, USA.
--->
+Copyright (c) 2022 PAL Robotics S.L. All rights reserved.
+Licensed under the Apache License, Version 2.0 (the "License");
+you may not use this file except in compliance with the License.
+You may obtain a copy of the License at
+    http://www.apache.org/licenses/LICENSE-2.0
+Unless required by applicable law or agreed to in writing, software
+distributed under the License is distributed on an "AS IS" BASIS,
+WITHOUT WARRANTIES OR CONDITIONS OF ANY KIND, either express or implied.
+See the License for the specific language governing permissions and
+limitations under the License.
+ -->
 <robot xmlns:xacro="http://ros.org/wiki/xacro">
   <!--External resources-->
@@ -30,7 +35,23 @@
   -->
   <xacro:macro name="hey5_hand" params="name parent reflect *origin">
+  <!-- Tool Link -->
+    <link name="${name}_tool_link">
+      <inertial>
+        <origin xyz="0 0 0" rpy="0 0 0" />
+        <mass value="0.0001" />
+        <inertia ixx="0.00001" ixy="0.0" ixz="0.0"
+                 iyy="0.00001" iyz="0.0"
+                 izz="0.00001" />
+      </inertial>
+    </link>
+    <joint name="${name}_tool_joint" type="fixed">
+      <xacro:insert_block name="origin"/>
+      <parent link="${parent}" />
+      <child link="${name}_tool_link" />
+       <axis xyz="0 0 0" />
+    </joint>
     <!--Palm-->
     <xacro:palm parent="${parent}" name="${name}_palm" reflect="${reflect}" >
-      <insert_block name="origin" />
+      <xacro:insert_block name="origin" />
     </xacro:palm>
     <!--Actuators-->

File: urdf/materials.urdf.xacro (robot description, xacro)
@@ -1,10 +1,15 @@
 <?xml version="1.0"?>
 <!--
-  Copyright (c) 2011, PAL Robotics, S.L.
-  All rights reserved.
-  This work is licensed under the Creative Commons Attribution 4.0 International License.
-  To view a copy of this license, visit http://creativecommons.org/licenses/by/4.0 or send a letter to
-  Creative Commons, 444 Castro Street, Suite 900, Mountain View, California, 94041, USA.
--->
+Copyright (c) 2022 PAL Robotics S.L. All rights reserved.
+Licensed under the Apache License, Version 2.0 (the "License");
+you may not use this file except in compliance with the License.
+You may obtain a copy of the License at
+    http://www.apache.org/licenses/LICENSE-2.0
+Unless required by applicable law or agreed to in writing, software
+distributed under the License is distributed on an "AS IS" BASIS,
+WITHOUT WARRANTIES OR CONDITIONS OF ANY KIND, either express or implied.
+See the License for the specific language governing permissions and
+limitations under the License.
+ -->
 <robot>
  <material name="Hey5DarkGrey">
